File: kicad/guitar_effect.kicad_sch (KiCad schematic)
At the start: 90 parts, among them J3 Header_1x5_male, Q2 MMBF5457, Q3 BC850C, Q4 BC850C, U1 USB_C, U2 OPA197IDBV, U3 OPA197IDBV, U4 78L05, U5 LM13700, U6 OPA197IDBV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

Commit message: Added bom
Parts:
- C11, C12: MIN_ORDER 0.0319 -> 20
Changed lines of the file:
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@@
       (effects (font (size 1.27 1.27)) hide)
     )
-    (property "MIN_ORDER" "0.0319" (at 167.64 144.78 0)
+    (property "MIN_ORDER" "20" (at 167.64 144.78 0)
       (effects (font (size 1.27 1.27)) hide)
     )
@@
       (effects (font (size 1.27 1.27)) hide)
     )
-    (property "MIN_ORDER" "0.0319" (at 104.14 144.78 0)
-      (effects (font (size 1.27 1.27)) hide)
-    )
+    (property "MIN_ORDER" "20" (at 104.14 144.78 0)
+      (effects (font (size 1.27 1.27)) hide)
+    )
